File: KiCAD/breakout.sch (KiCad schematic (older format))
At the start: 17 parts, among them J1 video_out, J2 audio_out, SW1 power, SW2 start, U1 PIC12F1572, X1 28.636Mhz

Commit message: travail sur software2
Parts:
- RV1: value 1K (paddle) -> 2K (paddle)
Changed lines of the file:
@@
 EESchema Schematic File Version 4
+LIBS:breakout-cache
 EELAYER 26 0
 EELAYER END
@@
 P 6700 4400
 F 0 "RV1" H 6631 4354 50  0000 R CNN
-F 1 "1K (paddle)" H 6631 4445 50  0000 R CNN
+F 1 "2K (paddle)" H 6631 4445 50  0000 R CNN
 F 2 "" H 6700 4400 50  0001 C CNN
 F 3 "" H 6700 4400 50  0001 C CNN

Commit message: Travail sur code
Parts:
- removed D1: 1N4148, symbol device:D_ALT
- R1: value 1k2 -> 1k
Connections:
- net video_y: now also R2.1
Changed lines of the file:
@@
 P 6150 2550
 F 0 "R1" V 6050 2550 50  0000 C CNN
-F 1 "1k2" V 6150 2550 50  0000 C CNN
+F 1 "1k" V 6150 2550 50  0000 C CNN
 F 2 "" V 6080 2550 50  0001 C CNN
 F 3 "" H 6150 2550 50  0001 C CNN
@@
 Text Label 6000 2550 2    50   ~ 0
 chroma
-Text Label 5700 2775 2    50   ~ 0
+Text Label 6000 2775 2    50   ~ 0
 video_y
 Text Label 6000 3025 2    50   ~ 0
 sync
 $Comp
-L device:D_ALT D1
-U 1 1 5C770167
-P 5850 2775
-F 0 "D1" H 5850 2875 50  0000 C CNN
-F 1 "1N4148" H 5875 2675 50  0000 C CNN
-F 2 "" H 5850 2775 50  0001 C CNN
-F 3 "" H 5850 2775 50  0001 C CNN
-	1    5850 2775
-	-1   0    0    1
-$EndComp
-$Comp
 L device:Battery BT1

Commit message: travail sur code
Parts:
- added C2, C3: 100nF, symbol device:C
- added C?: 220pF, symbol device:C
- added R7: 10K, symbol device:R
- added R8: 470, symbol device:R
- renumbered D2 to D1
Connections:
- wire segments 13 -> 30
Other:
- moved on the sheet: R4, SW2
Changed lines of the file:
@@
 U 1 1 5C76EC79
 P 5550 4450
-F 0 "U1" H 5550 4815 60  0000 C CNN
+F 0 "U1" H 5550 4800 60  0000 C CNN
 F 1 "PIC12F1572" H 5550 4725 39  0000 C CNN
 F 2 "" H 5550 4250 60  0001 C CNN
@@
 Text GLabel 6700 4250 1    50   Input ~ 0
 +5v
-Text GLabel 5100 4300 1    50   Input ~ 0
+Text GLabel 5100 3850 1    50   Input ~ 0
 +5v
 $Comp
@@
 L device:R R4
 U 1 1 5C76F3FB
-P 6050 3375
-F 0 "R4" V 5925 3375 50  0000 C CNN
-F 1 "10K" V 6050 3375 50  0000 C CNN
-F 2 "" V 5980 3375 50  0001 C CNN
-F 3 "" H 6050 3375 50  0001 C CNN
-	1    6050 3375
-	0    -1   -1   0
-$EndComp
-Wire Wire Line
-	6200 3375 6325 3375
+P 5975 3375
+F 0 "R4" V 6050 3400 50  0000 C CNN
+F 1 "10K" V 5975 3375 50  0000 C CNN
+F 2 "" V 5905 3375 50  0001 C CNN
+F 3 "" H 5975 3375 50  0001 C CNN
+	1    5975 3375
+	0    -1   -1   0
+$EndComp
 Wire Wire Line
 	6325 3375 6450 3375
 Connection ~ 6325 3375
-Text Label 5900 3375 2    50   ~ 0
+Text Label 5825 3375 2    50   ~ 0
 audio
 Text Label 6000 4500 0    50   ~ 0
@@
 L switches:SW_Push_45deg SW2
 U 1 1 5C76F596
-P 4950 4950
-F 0 "SW2" V 4996 4809 50  0000 R CNN
-F 1 "start" V 4900 4900 50  0000 R CNN
-F 2 "" H 4950 4950 50  0001 C CNN
-F 3 "" H 4950 4950 50  0001 C CNN
-	1    4950 4950
+P 4975 5125
+F 0 "SW2" V 5021 4984 50  0000 R CNN
+F 1 "start" V 4925 5075 50  0000 R CNN
+F 2 "" H 4975 5125 50  0001 C CNN
+F 3 "" H 4975 5125 50  0001 C CNN
+	1    4975 5125
 	0    -1   -1   0
 $EndComp
@@
 L power:GND #PWR09
 U 1 1 5C76F6D6
-P 4850 5050
-F 0 "#PWR09" H 4850 4800 50  0001 C CNN
-F 1 "GND" H 4855 4877 50  0000 C CNN
-F 2 "" H 4850 5050 50  0001 C CNN
-F 3 "" H 4850 5050 50  0001 C CNN
-	1    4850 5050
-	1    0    0    -1
-$EndComp
-Wire Wire Line
-	5050 4850 5050 4600
-Wire Wire Line
-	5050 4600 5100 4600
+P 4875 5325
+F 0 "#PWR09" H 4875 5075 50  0001 C CNN
+F 1 "GND" H 4880 5152 50  0000 C CNN
+F 2 "" H 4875 5325 50  0001 C CNN
+F 3 "" H 4875 5325 50  0001 C CNN
+	1    4875 5325
+	1    0    0    -1
+$EndComp
+Wire Wire Line
+	5050 4600 5075 4600
 $Comp
 L conn:Conn_Coaxial J1
@@
 $EndComp
 $Comp
-L device:D_ALT D2
+L device:D_ALT D1
 U 1 1 5C770637
 P 4400 3100
-F 0 "D2" H 4400 3200 50  0000 C CNN
+F 0 "D1" H 4400 3200 50  0000 C CNN
 F 1 "1N4001" H 4425 3000 50  0000 C CNN
 F 2 "" H 4400 3100 50  0001 C CNN
@@
 $EndComp
 NoConn ~ 4000 4400
+$Comp
+L device:R R7
+U 1 1 5C83F1D9
+P 4900 4600
+F 0 "R7" V 5000 4600 50  0000 C CNN
+F 1 "10K" V 4900 4575 50  0000 C CNN
+F 2 "" V 4830 4600 50  0001 C CNN
+F 3 "" H 4900 4600 50  0001 C CNN
+	1    4900 4600
+	0    1    1    0
+$EndComp
+Wire Wire Line
+	4750 4600 4750 4250
+Wire Wire Line
+	4750 4250 5100 4250
+Wire Wire Line
+	5100 4250 5100 4300
+$Comp
+L device:R R8
+U 1 1 5C83F7B0
+P 5075 4750
+F 0 "R8" V 5175 4750 50  0000 C CNN
+F 1 "470" V 5075 4725 50  0000 C CNN
+F 2 "" V 5005 4750 50  0001 C CNN
+F 3 "" H 5075 4750 50  0001 C CNN
+	1    5075 4750
+	1    0    0    -1
+$EndComp
+Connection ~ 5075 4600
+Wire Wire Line
+	5075 4600 5100 4600
+Wire Wire Line
+	5075 4900 5075 4950
+$Comp
+L device:C C2
+U 1 1 5C83FD1B
+P 5525 3925
+F 0 "C2" V 5475 4025 50  0000 C CNN
+F 1 "100nF" V 5575 4075 50  0000 C CNN
+F 2 "" H 5563 3775 50  0001 C CNN
+F 3 "" H 5525 3925 50  0001 C CNN
+	1    5525 3925
+	0    1    1    0
+$EndComp
+Wire Wire Line
+	5100 3850 5100 3925
+Connection ~ 5100 4250
+Wire Wire Line
+	5100 3925 5375 3925
+Connection ~ 5100 3925
+Wire Wire Line
+	5100 3925 5100 4250
+Wire Wire Line
+	5675 3925 6000 3925
+Wire Wire Line
+	6000 3925 6000 4100
+Connection ~ 6000 4100
+$Comp
+L device:C C3
+U 1 1 5C84052A
+P 5525 5100
+F 0 "C3" H 5350 5125 50  0000 C CNN
+F 1 "100nF" H 5400 5000 50  0000 C CNN
+F 2 "" H 5563 4950 50  0001 C CNN
+F 3 "" H 5525 5100 50  0001 C CNN
+	1    5525 5100
+	-1   0    0    1
+$EndComp
+Wire Wire Line
+	5525 4950 5075 4950
+Connection ~ 5075 4950
+Wire Wire Line
+	5075 4950 5075 5025
+Wire Wire Line
+	4875 5225 4875 5325
+Wire Wire Line
+	5525 5250 5525 5325
+Wire Wire Line
+	5525 5325 4875 5325
+Connection ~ 4875 5325
+$Comp
+L device:C C?
+U 1 1 5C840FAE
+P 6125 3525
+F 0 "C?" H 6275 3525 50  0000 C CNN
+F 1 "220pF" H 6275 3625 50  0000 C CNN
+F 2 "" H 6163 3375 50  0001 C CNN
+F 3 "" H 6125 3525 50  0001 C CNN
+	1    6125 3525
+	-1   0    0    1
+$EndComp
+Wire Wire Line
+	6200 3675 6325 3675
+Connection ~ 6325 3675
+Wire Wire Line
+	6125 3375 6325 3375
+Connection ~ 6125 3375
+Wire Wire Line
+	6200 3700 6200 3675
+Wire Wire Line
+	6200 3675 6125 3675
+Connection ~ 6200 3675
 $EndSCHEMATC

Commit message: travail sur code
Parts:
- removed X1: 28.636Mhz, Oscillators:Oscillator_SMD_Abracon_ASE-4pin_3.2x2.5mm, symbol Oscillators:ASE-xxxMHz
- added X1: 28.636Mhz, Oscillators:Oscillator_DIP-8, symbol Oscillators:CXO_DIP8
- C2, C3: value 100nF -> 220nF
- C4: renamed from C?; value 220pF -> 100pF
Connections:
- wire segments 30 -> 29
Other:
- moved on the sheet: R7
Changed lines of the file:
@@
-	1    0    0    -1
-$EndComp
-$Comp
-L Oscillators:ASE-xxxMHz X1
-U 1 1 5C76ED76
-P 4300 4400
-F 0 "X1" H 4525 4300 50  0000 L CNN
-F 1 "28.636Mhz" H 4350 4650 50  0000 L CNN
-F 2 "Oscillators:Oscillator_SMD_Abracon_ASE-4pin_3.2x2.5mm" H 5000 4050 50  0001 C CNN
-F 3 "http://www.abracon.com/Oscillators/ASV.pdf" H 4200 4400 50  0001 C CNN
-	1    4300 4400
 	1    0    0    -1
 $EndComp
@@
 	1    0    0    -1
 $EndComp
-Wire Wire Line
-	5050 4600 5075 4600
 $Comp
 L conn:Conn_Coaxial J1
@@
 L device:R R7
 U 1 1 5C83F1D9
-P 4900 4600
-F 0 "R7" V 5000 4600 50  0000 C CNN
-F 1 "10K" V 4900 4575 50  0000 C CNN
-F 2 "" V 4830 4600 50  0001 C CNN
-F 3 "" H 4900 4600 50  0001 C CNN
-	1    4900 4600
-	0    1    1    0
+P 4750 4750
+F 0 "R7" V 4850 4750 50  0000 C CNN
+F 1 "10K" V 4750 4725 50  0000 C CNN
+F 2 "" V 4680 4750 50  0001 C CNN
+F 3 "" H 4750 4750 50  0001 C CNN
+	1    4750 4750
+	-1   0    0    1
 $EndComp
 Wire Wire Line
@@
 	1    0    0    -1
 $EndComp
-Connection ~ 5075 4600
-Wire Wire Line
-	5075 4600 5100 4600
 Wire Wire Line
 	5075 4900 5075 4950
@@
 P 5525 3925
 F 0 "C2" V 5475 4025 50  0000 C CNN
-F 1 "100nF" V 5575 4075 50  0000 C CNN
+F 1 "220nF" V 5575 4075 50  0000 C CNN
 F 2 "" H 5563 3775 50  0001 C CNN
 F 3 "" H 5525 3925 50  0001 C CNN
@@
 P 5525 5100
 F 0 "C3" H 5350 5125 50  0000 C CNN
-F 1 "100nF" H 5400 5000 50  0000 C CNN
+F 1 "220nF" H 5400 5000 50  0000 C CNN
 F 2 "" H 5563 4950 50  0001 C CNN
 F 3 "" H 5525 5100 50  0001 C CNN
@@
 Connection ~ 4875 5325
 $Comp
-L device:C C?
+L device:C C4
 U 1 1 5C840FAE
 P 6125 3525
-F 0 "C?" H 6275 3525 50  0000 C CNN
-F 1 "220pF" H 6275 3625 50  0000 C CNN
+F 0 "C4" H 6275 3525 50  0000 C CNN
+F 1 "100pF" H 6275 3625 50  0000 C CNN
 F 2 "" H 6163 3375 50  0001 C CNN
 F 3 "" H 6125 3525 50  0001 C CNN
@@
 	-1   0    0    1
 $EndComp
-Wire Wire Line
-	6200 3675 6325 3675
 Connection ~ 6325 3675
 Wire Wire Line
 	6125 3375 6325 3375
 Connection ~ 6125 3375
-Wire Wire Line
-	6200 3700 6200 3675
-Wire Wire Line
-	6200 3675 6125 3675
-Connection ~ 6200 3675
+$Comp
+L Oscillators:CXO_DIP8 X1
+U 1 1 5C8529EE
+P 4300 4400
+F 0 "X1" H 4025 4675 50  0000 L CNN
+F 1 "28.636Mhz" H 4400 4650 50  0000 L CNN
+F 2 "Oscillators:Oscillator_DIP-8" H 4750 4050 50  0001 C CNN
+F 3 "http://cdn-reichelt.de/documents/datenblatt/B400/OSZI.pdf" H 4200 4400 50  0001 C CNN
+	1    4300 4400
+	1    0    0    -1
+$EndComp
+Wire Wire Line
+	4750 4900 4750 4950
+Wire Wire Line
+	4750 4950 5075 4950
+Wire Wire Line
+	5075 4600 5100 4600
+Wire Wire Line
+	6125 3675 6325 3675
 $EndSCHEMATC

Commit message: coding
Parts:
- C4: value 100pF -> 47nF
Changed lines of the file:
@@
 P 6125 3525
 F 0 "C4" H 6275 3525 50  0000 C CNN
-F 1 "100pF" H 6275 3625 50  0000 C CNN
+F 1 "47nF" H 6275 3625 50  0000 C CNN
 F 2 "" H 6163 3375 50  0001 C CNN
 F 3 "" H 6125 3525 50  0001 C CNN

Commit message: almost completed
Parts:
- added C5: 220nF, symbol device:C
- added R9: 150, symbol device:R
Connections:
- net +5v: now also R9.2; no longer RV1.3
- net GND: now also C5.1
- new net: C5.2, R9.1, RV1.3
Changed lines of the file:
@@
 	1    0    0    -1
 $EndComp
-Text GLabel 6700 4250 1    50   Input ~ 0
+Text GLabel 6700 3950 1    50   Input ~ 0
 +5v
 Text GLabel 5100 3850 1    50   Input ~ 0
@@
 P 6600 3575
 F 0 "#PWR04" H 6600 3325 50  0001 C CNN
-F 1 "GND" H 6605 3402 50  0000 C CNN
+F 1 "GND" H 6600 3450 50  0000 C CNN
 F 2 "" H 6600 3575 50  0001 C CNN
 F 3 "" H 6600 3575 50  0001 C CNN
@@
 Wire Wire Line
 	6125 3675 6325 3675
+$Comp
+L device:R R9
+U 1 1 5C8D60BE
+P 6700 4100
+F 0 "R9" V 6575 4100 50  0000 C CNN
+F 1 "150" V 6700 4100 50  0000 C CNN
+F 2 "" V 6630 4100 50  0001 C CNN
+F 3 "" H 6700 4100 50  0001 C CNN
+	1    6700 4100
+	-1   0    0    1
+$EndComp
+$Comp
+L device:C C5
+U 1 1 5C8D6341
+P 7250 4250
+F 0 "C5" V 7200 4350 50  0000 C CNN
+F 1 "220nF" V 7300 4400 50  0000 C CNN
+F 2 "" H 7288 4100 50  0001 C CNN
+F 3 "" H 7250 4250 50  0001 C CNN
+	1    7250 4250
+	0    1    1    0
+$EndComp
+Wire Wire Line
+	7100 4250 6700 4250
+Connection ~ 6700 4250
+$Comp
+L power:GND #PWR010
+U 1 1 5C8D6943
+P 7700 4250
+F 0 "#PWR010" H 7700 4000 50  0001 C CNN
+F 1 "GND" H 7705 4077 50  0000 C CNN
+F 2 "" H 7700 4250 50  0001 C CNN
+F 3 "" H 7700 4250 50  0001 C CNN
+	1    7700 4250
+	1    0    0    -1
+$EndComp
+Wire Wire Line
+	7400 4250 7700 4250
 $EndSCHEMATC
