File: KiCAD/ntsc-1575/_saved_ntsc-1575.sch (KiCad schematic (older format))
At the start: 43 parts, among them J1 video_out, J2 audio_out, SW1 power, SW2 start, SW3 UP, SW4 DOWN, SW5 BTN_A, SW6 LEFT, SW7 BTN_B, SW8 RIGHT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

Commit message: travail sur ntsc-1575.X ajout est color bars
Parts:
- removed C1, C7: 100n, symbol device:C
- C5: renamed from C6; value 100nF -> 220nF
- renumbered C2 to C1, C3 to C2, C4 to C3, C5 to C4, C8 to C6, C9 to C7
Connections:
- net chroma0: now also R1.2
Other:
- moved on the sheet: D2, D3, D4, D5, D6, D7, SW3A, SW4A, SW5A, SW6A, SW7A, SW8A
